Commit message: Now with all the models

File: urdf/test.xacro (robot description, xacro)
@@ -61,5 +61,5 @@
       <origin xyz="0 0 0" rpy="0 0 0"/>
       <geometry>
-        <mesh filename="package://rrbot_description/meshes/hokuyo.dae"/>
+        <mesh filename="package://beginner_tutorials/models/hokuyo.dae"/>
       </geometry>
     </visual>

Commit message: Ordenando algo mas el asunto

File: urdf/test.xacro (robot description, xacro)
@@ -12,5 +12,5 @@
   <xacro:property name="axel_offset" value="0.05" />
   <!-- Import all Gazebo-customization elements, including Gazebo colors -->
-  <xacro:include filename="$(find beginner_tutorials)/urdf/test.gazebo" />
+  <xacro:include filename="$(find sonar_sim)/urdf/test.gazebo" />
   <!-- Used for fixing robot to Gazebo 'base_link' -->
   <link name="world"/>
@@ -61,5 +61,5 @@
       <origin xyz="0 0 0" rpy="0 0 0"/>
       <geometry>
-        <mesh filename="package://beginner_tutorials/models/hokuyo.dae"/>
+        <mesh filename="package://sonar_sim/models/hokuyo.dae"/>
       </geometry>
     </visual>
